Commit message: fine parte 4

File: arm_description/urdf/arm.urdf.xacro (robot description, xacro)
@@ -4,4 +4,12 @@
     <color rgba="1 0 0 1"/>
   </material>
+  <link name="world">
+    <origin rpy="0 0 0" xyz="0 0 0"/>
+  </link>
+  <joint name="arm_base_joint" type="fixed">
+      <origin rpy="0.0 0 0" xyz="0 0 0"/>
+      <parent link="world"/>
+      <child link="base_link"/>
+  </joint>
   <link name="base_link">
     <visual>
@@ -348,4 +356,33 @@
     </inertial>
   </link>
+<!-- added camera link -->
+ <link name="camera_link">
+    <visual>
+      <geometry>
+        <box size='0.05 0.05 0.05'/>
+      </geometry>
+      <origin rpy="0 0 0" xyz="0 0 0.02"/>
+      <material name="yellow">
+        <color rgba="1 1 0 1"/>
+      </material>
+    </visual>
+      <collision>
+        <geometry>
+          <box size='0.05 0.05 0.05'/>
+        </geometry>
+        <origin rpy="0 0 0" xyz="0 0 0"/>
+      </collision>
+    <inertial>
+      <origin xyz="0 0 0" rpy="0 0 0"/>
+      <mass value="0.2"/>
+      <inertia ixx="3.3e-05" ixy="0.0" ixz="0.0" iyy="5.8e-05" iyz="0.0" izz="4.1e-05"/>
+    </inertial>
+  </link>
+  <!-- added  camera joint -->
+  <joint name="camera_joint" type="fixed">
+      <parent link="base_link"/>
+      <child link="camera_link"/>
+      <origin xyz="0 0 0" rpy="0 0 0"/>
+  </joint>
   <gazebo>
     <plugin filename="ign_ros2_control-system" name="ign_ros2_control::IgnitionROS2ControlPlugin">
@@ -354,9 +391,17 @@
     </plugin>
   </gazebo>
+  <gazebo>
+	  <plugin filename="gz-sim-sensors-system"
+		name="gz::sim::systems::Sensors">
+		<render_engine>ogre2</render_engine>
+	 </plugin>
+  </gazebo>
   <xacro:include filename="$(find arm_description)/urdf/arm_hardware_interface.xacro"/>
+  <xacro:include filename="$(find arm_gazebo)/urdf/arm_camera.xacro"/>
+  <xacro:arm_camera link="camera_link"/>
   <ros2_control name="HardwareInterface_Ignition" type="system">
      <hardware>
       <plugin>ign_ros2_control/IgnitionSystem</plugin>
-    </hardware>
+     </hardware>
     <xacro:PositionJointInterface name="j0" initial_pos="0.0"/>
     <xacro:PositionJointInterface name="j1" initial_pos="0.0"/>

Commit message: fine parte opzionale

File: arm_description/urdf/arm.urdf.xacro (robot description, xacro)
@@ -357,5 +357,5 @@
   </link>
 <!-- added camera link -->
- <link name="camera_link">
+ <!-- <link name="camera_link">
     <visual>
       <geometry>
@@ -378,11 +378,14 @@
       <inertia ixx="3.3e-05" ixy="0.0" ixz="0.0" iyy="5.8e-05" iyz="0.0" izz="4.1e-05"/>
     </inertial>
-  </link>
+  </link> -->
   <!-- added  camera joint -->
-  <joint name="camera_joint" type="fixed">
+  <!-- <joint name="camera_joint" type="fixed">
       <parent link="base_link"/>
       <child link="camera_link"/>
       <origin xyz="0 0 0" rpy="0 0 0"/>
   </joint>
+ -->
+  <xacro:include filename="$(find arm_gazebo)/urdf/camera.xacro"/>
+  <xacro:camera parent="base_link" child="camera_link"/>
   <gazebo>
     <plugin filename="ign_ros2_control-system" name="ign_ros2_control::IgnitionROS2ControlPlugin">
@@ -398,6 +401,7 @@
   </gazebo>
   <xacro:include filename="$(find arm_description)/urdf/arm_hardware_interface.xacro"/>
-  <xacro:include filename="$(find arm_gazebo)/urdf/arm_camera.xacro"/>
+  <!-- <xacro:include filename="$(find arm_gazebo)/urdf/arm_camera.xacro"/>
   <xacro:arm_camera link="camera_link"/>
+   -->
   <ros2_control name="HardwareInterface_Ignition" type="system">
      <hardware>

File: arm_gazebo/urdf/camera.xacro (robot description, xacro)
@@ -1,7 +1,7 @@
 <?xml version="1.0" encoding="utf-8"?>
 <robot xmlns:xacro="http://www.ros.org/wiki/xacro">
-<xacro:macro name="camera" params="name_camera_link name_joint ">
+<xacro:macro name="camera" params=" parent child ">
     <!-- added camera link -->
-    <link name="${name_camera_link}">
+    <link name="camera_link">
         <visual>
         <geometry>
@@ -26,9 +26,11 @@
     </link>
     <!-- added  camera joint -->
-    <joint name="${name_joint}" type="fixed">
-        <parent link="base_link"/>
-        <child link="${name_camera}"/>
+    <joint name="camera_joint" type="fixed">
+        <parent link="${parent}"/>
+        <child link="${child}"/>
         <origin xyz="0 0 0" rpy="0 0 0"/>
     </joint>
+    <xacro:include filename="$(find arm_gazebo)/urdf/arm_camera.xacro"/>
+    <xacro:arm_camera link="camera_link"/>
 </xacro:macro>
 </robot>

Commit message: fine tutto

File: arm_description/urdf/arm.urdf.xacro (robot description, xacro)
@@ -356,34 +356,4 @@
     </inertial>
   </link>
-<!-- added camera link -->
- <!-- <link name="camera_link">
-    <visual>
-      <geometry>
-        <box size='0.05 0.05 0.05'/>
-      </geometry>
-      <origin rpy="0 0 0" xyz="0 0 0.02"/>
-      <material name="yellow">
-        <color rgba="1 1 0 1"/>
-      </material>
-    </visual>
-      <collision>
-        <geometry>
-          <box size='0.05 0.05 0.05'/>
-        </geometry>
-        <origin rpy="0 0 0" xyz="0 0 0"/>
-      </collision>
-    <inertial>
-      <origin xyz="0 0 0" rpy="0 0 0"/>
-      <mass value="0.2"/>
-      <inertia ixx="3.3e-05" ixy="0.0" ixz="0.0" iyy="5.8e-05" iyz="0.0" izz="4.1e-05"/>
-    </inertial>
-  </link> -->
-  <!-- added  camera joint -->
-  <!-- <joint name="camera_joint" type="fixed">
-      <parent link="base_link"/>
-      <child link="camera_link"/>
-      <origin xyz="0 0 0" rpy="0 0 0"/>
-  </joint>
- -->
   <xacro:include filename="$(find arm_gazebo)/urdf/camera.xacro"/>
   <xacro:camera parent="base_link" child="camera_link"/>
@@ -401,7 +371,4 @@
   </gazebo>
   <xacro:include filename="$(find arm_description)/urdf/arm_hardware_interface.xacro"/>
-  <!-- <xacro:include filename="$(find arm_gazebo)/urdf/arm_camera.xacro"/>
-  <xacro:arm_camera link="camera_link"/>
-   -->
   <ros2_control name="HardwareInterface_Ignition" type="system">
      <hardware>

Commit message: risolto tutto

File: arm_description/urdf/arm.urdf.xacro (robot description, xacro)
@@ -4,8 +4,6 @@
     <color rgba="1 0 0 1"/>
   </material>
-  <link name="world">
-    <origin rpy="0 0 0" xyz="0 0 0"/>
-  </link>
-  <joint name="arm_base_joint" type="fixed">
+  <link name="world"/>
+  <joint name="iiwa_base_joint" type="fixed">
       <origin rpy="0.0 0 0" xyz="0 0 0"/>
       <parent link="world"/>
@@ -356,6 +354,31 @@
     </inertial>
   </link>
-  <xacro:include filename="$(find arm_gazebo)/urdf/camera.xacro"/>
-  <xacro:camera parent="base_link" child="camera_link"/>
+<link name="camera_link">
+    <visual>
+      <geometry>
+        <box size='0.05 0.05 0.05'/>
+      </geometry>
+      <origin rpy="0 0 0" xyz="0 0 0.02"/>
+      <material name="yellow">
+        <color rgba="1 1 0 1"/>
+      </material>
+    </visual>
+      <collision>
+        <geometry>
+          <box size='0.05 0.05 0.05'/>
+        </geometry>
+        <origin rpy="0 0 0" xyz="0 0 0"/>
+      </collision>
+    <inertial>
+      <origin xyz="0 0 0" rpy="0 0 0"/>
+      <mass value="0.2"/>
+      <inertia ixx="3.3e-05" ixy="0.0" ixz="0.0" iyy="5.8e-05" iyz="0.0" izz="4.1e-05"/>
+    </inertial>
+  </link>
+  <joint name="camera_joint" type="fixed">
+      <parent link="base_link"/>
+      <child link="camera_link"/>
+      <origin xyz="0 0 0" rpy="0 0 0"/>
+  </joint>
   <gazebo>
     <plugin filename="ign_ros2_control-system" name="ign_ros2_control::IgnitionROS2ControlPlugin">
@@ -364,15 +387,10 @@
     </plugin>
   </gazebo>
-  <gazebo>
-	  <plugin filename="gz-sim-sensors-system"
-		name="gz::sim::systems::Sensors">
-		<render_engine>ogre2</render_engine>
-	 </plugin>
-  </gazebo>
   <xacro:include filename="$(find arm_description)/urdf/arm_hardware_interface.xacro"/>
+  <xacro:include filename="$(find arm_gazebo)/urdf/arm_camera.xacro"/>
   <ros2_control name="HardwareInterface_Ignition" type="system">
-     <hardware>
+    <hardware>
       <plugin>ign_ros2_control/IgnitionSystem</plugin>
-     </hardware>
+    </hardware>
     <xacro:PositionJointInterface name="j0" initial_pos="0.0"/>
     <xacro:PositionJointInterface name="j1" initial_pos="0.0"/>
@@ -380,3 +398,10 @@
     <xacro:PositionJointInterface name="j3" initial_pos="0.0"/>
   </ros2_control>
+  <gazebo>
+	  <plugin filename="gz-sim-sensors-system"
+		name="gz::sim::systems::Sensors">
+	  <render_engine>ogre2</render_engine>
+	  </plugin>
+   </gazebo>
+  <xacro:arm_camera link="camera_link"/>
 </robot>
